File: hardware/arduino_pir_sensor.brd (EAGLE design)
At the start: 69 x 34.8 mm, 43 parts, among them U2 TPS61097-33, U3 BISS0001SO16, U4 NRF24L01+_MODULE, U5 D203S

Commit message: - cutout in ground planes on all PCB layers added below wireless module antenna - serial communication connector added
Parts:
- added JP1: (no value), endy-connectors:1X03
- moved C16 2.70 mm to (25.9, 18.5), turned to 270 degrees
- moved U4 1.78 mm to (29.2, 5.71)
Connections:
- net GND: now also JP1.3
- net RXI: now also JP1.2
- net TXO: now also JP1.1
Routing:
- net RXI: track 0.00 -> 20.9 mm, vias 0 -> 1
- net RESET: track 56.1 -> 36.4 mm, vias 1 -> 2
- net TXO: track 0.00 -> 17.9 mm, vias 0 -> 1
- net 3.3V: track 201.0 -> 206.3 mm
- net A0: track 77.1 -> 73.2 mm
- net D9: track 34.9 -> 33.1 mm
- net D10: track 40.4 -> 38.8 mm
- net SCK: track 36.0 -> 34.6 mm
- net MISO: track 28.9 -> 27.8 mm
- net MOSI: track 39.4 -> 38.4 mm
- net N$17: track 7.53 -> 8.25 mm
Other:
- board text added: "GND"
- board text added: "RXI"
- board text added: "TXO"
